File: board/22-ELC-1-01-R1 (TSCU)/CAN_controller_transceiver.kicad_sch (KiCad schematic)
At the start: 15 parts, among them U1 MCP2515-xSO, U2 SN65HVD230, Y1 16 MHz

Commit message: Finalized schematic, started board layout
Parts:
- C2, C3, C4, C5: footprint Capacitor_SMD:C_0603_1608Metric_Pad1.08x0.95mm_HandSolder -> Capacitor_SMD:C_0402_1005Metric
- R4, R5: footprint Resistor_SMD:R_0603_1608Metric_Pad0.98x0.95mm_HandSolder -> FixedTextSizes:R_0402_1005Metric
Changed lines of the file:
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@@
       (effects (font (size 1.27 1.27)) (justify left))
     )
-    (property "Footprint" "Capacitor_SMD:C_0603_1608Metric_Pad1.08x0.95mm_HandSolder" (id 2) (at 152.4 92.71 0)
+    (property "Footprint" "Capacitor_SMD:C_0402_1005Metric" (id 2) (at 152.4 92.71 0)
       (effects (font (size 1.27 1.27)) hide)
     )
@@
   (symbol (lib_id "power:GND") (at 148.59 118.11 0) (unit 1)
     (in_bom yes) (on_board yes)
-    (property "Reference" "#PWR029" (id 0) (at 148.59 124.46 0)
+    (property "Reference" "#PWR028" (id 0) (at 148.59 124.46 0)
       (effects (font (size 1.27 1.27)) hide)
     )
@@
   (symbol (lib_id "power:GND") (at 157.48 93.98 0) (unit 1)
     (in_bom yes) (on_board yes)
-    (property "Reference" "#PWR030" (id 0) (at 157.48 100.33 0)
+    (property "Reference" "#PWR029" (id 0) (at 157.48 100.33 0)
       (effects (font (size 1.27 1.27)) hide)
     )
@@
   (symbol (lib_id "power:GND") (at 132.08 113.03 270) (unit 1)
     (in_bom yes) (on_board yes)
-    (property "Reference" "#PWR027" (id 0) (at 125.73 113.03 0)
+    (property "Reference" "#PWR026" (id 0) (at 125.73 113.03 0)
       (effects (font (size 1.27 1.27)) hide)
     )
@@
   (symbol (lib_id "power:GND") (at 83.82 139.7 0) (unit 1)
     (in_bom yes) (on_board yes)
-    (property "Reference" "#PWR023" (id 0) (at 83.82 146.05 0)
+    (property "Reference" "#PWR022" (id 0) (at 83.82 146.05 0)
       (effects (font (size 1.27 1.27)) hide)
     )
@@
   (symbol (lib_id "power:GND") (at 45.72 125.73 0) (unit 1)
     (in_bom yes) (on_board yes)
-    (property "Reference" "#PWR019" (id 0) (at 45.72 132.08 0)
+    (property "Reference" "#PWR018" (id 0) (at 45.72 132.08 0)
       (effects (font (size 1.27 1.27)) hide)
     )
@@
   (symbol (lib_id "power:GND") (at 55.88 125.73 0) (unit 1)
     (in_bom yes) (on_board yes)
-    (property "Reference" "#PWR020" (id 0) (at 55.88 132.08 0)
+    (property "Reference" "#PWR019" (id 0) (at 55.88 132.08 0)
       (effects (font (size 1.27 1.27)) hide)
     )
@@
     (property "Reference" "C2" (id 0) (at 37.465 120.015 0))
     (property "Value" "22pf" (id 1) (at 40.005 125.095 0))
-    (property "Footprint" "Capacitor_SMD:C_0603_1608Metric_Pad1.08x0.95mm_HandSolder" (id 2) (at 36.83 123.19 0)
+    (property "Footprint" "Capacitor_SMD:C_0402_1005Metric" (id 2) (at 36.83 123.19 0)
       (effects (font (size 1.27 1.27)) hide)
     )
@@
     (property "Reference" "C3" (id 0) (at 37.465 132.08 0))
     (property "Value" "22pf" (id 1) (at 40.005 127 0))
-    (property "Footprint" "Capacitor_SMD:C_0603_1608Metric_Pad1.08x0.95mm_HandSolder" (id 2) (at 36.83 128.27 0)
+    (property "Footprint" "Capacitor_SMD:C_0402_1005Metric" (id 2) (at 36.83 128.27 0)
       (effects (font (size 1.27 1.27)) hide)
     )
@@
   (symbol (lib_id "power:GND") (at 31.75 125.73 0) (unit 1)
     (in_bom yes) (on_board yes)
-    (property "Reference" "#PWR018" (id 0) (at 31.75 132.08 0)
+    (property "Reference" "#PWR017" (id 0) (at 31.75 132.08 0)
       (effects (font (size 1.27 1.27)) hide)
     )
@@
       (effects (font (size 1.27 1.27)) (justify left))
     )
-    (property "Footprint" "Capacitor_SMD:C_0603_1608Metric_Pad1.08x0.95mm_HandSolder" (id 2) (at 87.63 92.71 0)
+    (property "Footprint" "Capacitor_SMD:C_0402_1005Metric" (id 2) (at 87.63 92.71 0)
       (effects (font (size 1.27 1.27)) hide)
     )
@@
   (symbol (lib_id "power:GND") (at 92.71 93.98 0) (unit 1)
     (in_bom yes) (on_board yes)
-    (property "Reference" "#PWR024" (id 0) (at 92.71 100.33 0)
+    (property "Reference" "#PWR023" (id 0) (at 92.71 100.33 0)
       (effects (font (size 1.27 1.27)) hide)
     )
@@
   (symbol (lib_id "power:+5V") (at 148.59 91.44 0) (unit 1)
     (in_bom yes) (on_board yes)
-    (property "Reference" "#PWR028" (id 0) (at 148.59 95.25 0)
+    (property "Reference" "#PWR027" (id 0) (at 148.59 95.25 0)
       (effects (font (size 1.27 1.27)) hide)
     )
@@
   (symbol (lib_id "power:+5V") (at 132.08 110.49 90) (unit 1)
     (in_bom yes) (on_board yes)
-    (property "Reference" "#PWR026" (id 0) (at 135.89 110.49 0)
+    (property "Reference" "#PWR025" (id 0) (at 135.89 110.49 0)
       (effects (font (size 1.27 1.27)) hide)
     )
@@
   (symbol (lib_id "power:+5V") (at 83.82 90.17 0) (unit 1)
     (in_bom yes) (on_board yes)
-    (property "Reference" "#PWR022" (id 0) (at 83.82 93.98 0)
+    (property "Reference" "#PWR021" (id 0) (at 83.82 93.98 0)
       (effects (font (size 1.27 1.27)) hide)
     )
@@
       (effects (font (size 1.27 1.27)) (justify left))
     )
-    (property "Footprint" "Resistor_SMD:R_0603_1608Metric_Pad0.98x0.95mm_HandSolder" (id 2) (at 55.372 91.44 90)
+    (property "Footprint" "FixedTextSizes:R_0402_1005Metric" (id 2) (at 55.372 91.44 90)
       (effects (font (size 1.27 1.27)) hide)
     )
@@
   (symbol (lib_id "power:+5V") (at 57.15 87.63 0) (unit 1)
     (in_bom yes) (on_board yes)
-    (property "Reference" "#PWR021" (id 0) (at 57.15 91.44 0)
+    (property "Reference" "#PWR020" (id 0) (at 57.15 91.44 0)
       (effects (font (size 1.27 1.27)) hide)
     )
@@
   (symbol (lib_id "power:+5V") (at 109.22 125.73 0) (unit 1)
     (in_bom yes) (on_board yes)
-    (property "Reference" "#PWR025" (id 0) (at 109.22 129.54 0)
+    (property "Reference" "#PWR024" (id 0) (at 109.22 129.54 0)
       (effects (font (size 1.27 1.27)) hide)
     )
@@
       (effects (font (size 1.27 1.27)) (justify left))
     )
-    (property "Footprint" "Resistor_SMD:R_0603_1608Metric_Pad0.98x0.95mm_HandSolder" (id 2) (at 107.442 129.54 90)
-      (effects (font (size 1.27 1.27)) hide)
-    )
+    (property "Footprint" "FixedTextSizes:R_0402_1005Metric" (id 2) (at 107.442 129.54 90)
+      (effects (font (size 1.27 1.27)) hide)
+    )

Commit message: More progress
Parts:
- C2, C3, C4, C5: footprint Capacitor_SMD:C_0402_1005Metric -> FixedTextSizes:C_0402_1005Metric_Pad0.74x0.62mm_HandSolder_Reasonable_Text_Size
Changed lines of the file:
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@@
       (effects (font (size 1.27 1.27)) (justify left))
     )
-    (property "Footprint" "Capacitor_SMD:C_0402_1005Metric" (id 2) (at 152.4 92.71 0)
+    (property "Footprint" "FixedTextSizes:C_0402_1005Metric_Pad0.74x0.62mm_HandSolder_Reasonable_Text_Size" (id 2) (at 152.4 92.71 0)
       (effects (font (size 1.27 1.27)) hide)
     )
@@
   (symbol (lib_id "power:GND") (at 148.59 118.11 0) (unit 1)
     (in_bom yes) (on_board yes)
-    (property "Reference" "#PWR028" (id 0) (at 148.59 124.46 0)
+    (property "Reference" "#PWR031" (id 0) (at 148.59 124.46 0)
       (effects (font (size 1.27 1.27)) hide)
     )
@@
   (symbol (lib_id "power:GND") (at 157.48 93.98 0) (unit 1)
     (in_bom yes) (on_board yes)
-    (property "Reference" "#PWR029" (id 0) (at 157.48 100.33 0)
+    (property "Reference" "#PWR032" (id 0) (at 157.48 100.33 0)
       (effects (font (size 1.27 1.27)) hide)
     )
@@
   (symbol (lib_id "power:GND") (at 132.08 113.03 270) (unit 1)
     (in_bom yes) (on_board yes)
-    (property "Reference" "#PWR026" (id 0) (at 125.73 113.03 0)
+    (property "Reference" "#PWR029" (id 0) (at 125.73 113.03 0)
       (effects (font (size 1.27 1.27)) hide)
     )
@@
   (symbol (lib_id "power:GND") (at 83.82 139.7 0) (unit 1)
     (in_bom yes) (on_board yes)
-    (property "Reference" "#PWR022" (id 0) (at 83.82 146.05 0)
+    (property "Reference" "#PWR025" (id 0) (at 83.82 146.05 0)
       (effects (font (size 1.27 1.27)) hide)
     )
@@
   (symbol (lib_id "power:GND") (at 45.72 125.73 0) (unit 1)
     (in_bom yes) (on_board yes)
-    (property "Reference" "#PWR018" (id 0) (at 45.72 132.08 0)
+    (property "Reference" "#PWR021" (id 0) (at 45.72 132.08 0)
       (effects (font (size 1.27 1.27)) hide)
     )
@@
   (symbol (lib_id "power:GND") (at 55.88 125.73 0) (unit 1)
     (in_bom yes) (on_board yes)
-    (property "Reference" "#PWR019" (id 0) (at 55.88 132.08 0)
+    (property "Reference" "#PWR022" (id 0) (at 55.88 132.08 0)
       (effects (font (size 1.27 1.27)) hide)
     )
@@
     (property "Reference" "C2" (id 0) (at 37.465 120.015 0))
     (property "Value" "22pf" (id 1) (at 40.005 125.095 0))
-    (property "Footprint" "Capacitor_SMD:C_0402_1005Metric" (id 2) (at 36.83 123.19 0)
+    (property "Footprint" "FixedTextSizes:C_0402_1005Metric_Pad0.74x0.62mm_HandSolder_Reasonable_Text_Size" (id 2) (at 36.83 123.19 0)
       (effects (font (size 1.27 1.27)) hide)
     )
@@
     (property "Reference" "C3" (id 0) (at 37.465 132.08 0))
     (property "Value" "22pf" (id 1) (at 40.005 127 0))
-    (property "Footprint" "Capacitor_SMD:C_0402_1005Metric" (id 2) (at 36.83 128.27 0)
+    (property "Footprint" "FixedTextSizes:C_0402_1005Metric_Pad0.74x0.62mm_HandSolder_Reasonable_Text_Size" (id 2) (at 36.83 128.27 0)
       (effects (font (size 1.27 1.27)) hide)
     )
@@
   (symbol (lib_id "power:GND") (at 31.75 125.73 0) (unit 1)
     (in_bom yes) (on_board yes)
-    (property "Reference" "#PWR017" (id 0) (at 31.75 132.08 0)
+    (property "Reference" "#PWR020" (id 0) (at 31.75 132.08 0)
       (effects (font (size 1.27 1.27)) hide)
     )
@@
       (effects (font (size 1.27 1.27)) (justify left))
     )
-    (property "Footprint" "Capacitor_SMD:C_0402_1005Metric" (id 2) (at 87.63 92.71 0)
+    (property "Footprint" "FixedTextSizes:C_0402_1005Metric_Pad0.74x0.62mm_HandSolder_Reasonable_Text_Size" (id 2) (at 87.63 92.71 0)
       (effects (font (size 1.27 1.27)) hide)
     )
@@
   (symbol (lib_id "power:GND") (at 92.71 93.98 0) (unit 1)
     (in_bom yes) (on_board yes)
-    (property "Reference" "#PWR023" (id 0) (at 92.71 100.33 0)
+    (property "Reference" "#PWR026" (id 0) (at 92.71 100.33 0)
       (effects (font (size 1.27 1.27)) hide)
     )
@@
   (symbol (lib_id "power:+5V") (at 148.59 91.44 0) (unit 1)
     (in_bom yes) (on_board yes)
-    (property "Reference" "#PWR027" (id 0) (at 148.59 95.25 0)
+    (property "Reference" "#PWR030" (id 0) (at 148.59 95.25 0)
       (effects (font (size 1.27 1.27)) hide)
     )
@@
   (symbol (lib_id "power:+5V") (at 132.08 110.49 90) (unit 1)
     (in_bom yes) (on_board yes)
-    (property "Reference" "#PWR025" (id 0) (at 135.89 110.49 0)
+    (property "Reference" "#PWR028" (id 0) (at 135.89 110.49 0)
       (effects (font (size 1.27 1.27)) hide)
     )
@@
   (symbol (lib_id "power:+5V") (at 83.82 90.17 0) (unit 1)
     (in_bom yes) (on_board yes)
-    (property "Reference" "#PWR021" (id 0) (at 83.82 93.98 0)
+    (property "Reference" "#PWR024" (id 0) (at 83.82 93.98 0)
       (effects (font (size 1.27 1.27)) hide)
     )
@@
   (symbol (lib_id "power:+5V") (at 57.15 87.63 0) (unit 1)
     (in_bom yes) (on_board yes)
-    (property "Reference" "#PWR020" (id 0) (at 57.15 91.44 0)
+    (property "Reference" "#PWR023" (id 0) (at 57.15 91.44 0)
       (effects (font (size 1.27 1.27)) hide)
     )
@@
   (symbol (lib_id "power:+5V") (at 109.22 125.73 0) (unit 1)
     (in_bom yes) (on_board yes)
-    (property "Reference" "#PWR024" (id 0) (at 109.22 129.54 0)
-      (effects (font (size 1.27 1.27)) hide)
-    )
+    (property "Reference" "#PWR027" (id 0) (at 109.22 129.54 0)
+      (effects (font (size 1.27 1.27)) hide)
+    )
