File: board/22-ELC-1-01-R1 (TSCU)/20-ELC-1-01-R1.kicad_pcb (KiCad board)
At the start: 2 copper layers, 234 parts, among them J1 Conn_01x116, J10 Conn_01x01, J11 Conn_01x02, J12 Conn_01x02, J13 SWD, J2 Conn_01x02_Female, J3 Conn_01x06, J4 Conn_01x02, J5 Conn_01x02, J6 Conn_01x06, J7 Conn_01x01, J8 Conn_02x02_Counter_Clockwise, J9 Conn_02x02_Counter_Clockwise, Q1 AO3400A, Q10 AO3400A, Q11 SUD50P04-09L-E3, Q12 SUD50P04-09L-E3, Q2 2N7002, Q3 CSD18540Q5B, Q4 AO3400A, Q5 AO3400A, Q6 AO3400A, Q7 AO3400A, Q8 Q_NMOS_DGS, Q9 AO3400A, SW1 FAULT_RESET, SW2 SW_SPDT, U1 MCP2515-xSO, U10 ACPL-C79B, U11 LM358, U12 LM358, U13 LM358, U14 LM358, U15 STM32F105RCTx, U16 SN65HVD230, U17 SN65HVD230, U18 AMS1117-3.3, U2 SN65HVD230, U3 74AUC1G17, U4 LM393, U5 74HC08_2AND, U6 TPS5430DDA, U7 74HC74D,653, U8 SGM809-SXN3/TR, U9 RFMM-0505S, X1 placeholder_for_picture, X2 placeholder_for_picture, Y1 16 MHz, Y2 16MHz

Commit message: Finalized schematic, started board layout
Parts:
- removed the D18 at (130.5, 85.0)
- removed J12: Conn_01x02, Connector_PinHeader_2.54mm:PinHeader_1x02_P2.54mm_Vertical
- added C38: 10uF, Capacitor_SMD:C_0402_1005Metric, F.Cu at (223.5, 137.2)
- added C39: 10uF, Capacitor_SMD:C_0402_1005Metric, F.Cu at (230.3, 130.4)
- added C40: 100nF, Capacitor_SMD:C_0402_1005Metric, F.Cu at (230.3, 132.9)
- added C41: 100nF, Capacitor_SMD:C_0402_1005Metric, F.Cu at (234.6, 130.4)
- added C42: 22uF, Capacitor_SMD:C_0402_1005Metric, F.Cu at (225.9, 132.9)
- added C43: 22uF, Capacitor_SMD:C_0402_1005Metric, F.Cu at (225.9, 130.4)
- added D17: DT1446-04TS-7, Global Libraries:SOT95P280X100-6N, F.Cu at (72.9, 90.4)
- added D19: 20V, Diode_SMD:D_0603_1608Metric_Pad1.05x0.95mm_HandSolder, F.Cu at (246.8, 133.0)
- added D20: 0.7dV, Diode_SMD:D_0603_1608Metric_Pad1.05x0.95mm_HandSolder, F.Cu at (246.8, 130.4)
- added F2: 2A, Fuse:Fuse_0603_1608Metric_Pad1.05x0.95mm_HandSolder, F.Cu at (251.1, 130.4)
- added L2: 4u7, Inductor_SMD:L_Sunlord_MWSA0518_5.4x5.2mm, F.Cu at (220.0, 132.5)
- added PWR_3V1: LED, LED_SMD:LED_0603_1608Metric_Pad1.05x0.95mm_HandSolder, F.Cu at (242.4, 133.0)
- added PWR_5V1: 100, Resistor_SMD:R_0201_0603Metric_Pad0.64x0.40mm_HandSolder, F.Cu at (246.0, 135.2)
- added PWR_IN1: LED, LED_SMD:LED_0603_1608Metric_Pad1.05x0.95mm_HandSolder, F.Cu at (242.4, 130.4)
- added PWR_IN2: LED, LED_SMD:LED_0603_1608Metric_Pad1.05x0.95mm_HandSolder, F.Cu at (242.4, 135.6)
- added R72: 470, FixedTextSizes:R_0402_1005Metric, F.Cu at (250.4, 132.5)
- added R73: 0, FixedTextSizes:R_0402_1005Metric, F.Cu at (250.4, 134.3)
- added R74: 10K, FixedTextSizes:R_0402_1005Metric, F.Cu at (227.9, 135.4)
- added R75: 10K, FixedTextSizes:R_0402_1005Metric, F.Cu at (234.6, 132.9)
- added R76: 54.9K, FixedTextSizes:R_0402_1005Metric, F.Cu at (223.5, 139.7)
- C1, C10, C11, C12, C2, C3, C4, C5, C6, C7, C9: footprint Capacitor_SMD:C_0603_1608Metric_Pad1.08x0.95mm_HandSolder -> Capacitor_SMD:C_0402_1005Metric
- C13: renamed from C20; footprint Capacitor_SMD:C_0603_1608Metric_Pad1.08x0.95mm_HandSolder -> Capacitor_SMD:C_0402_1005Metric
- C14: renamed from C21; footprint Capacitor_SMD:C_0603_1608Metric_Pad1.08x0.95mm_HandSolder -> Capacitor_SMD:C_0402_1005Metric
- C15: renamed from C22; footprint Capacitor_SMD:C_0603_1608Metric_Pad1.08x0.95mm_HandSolder -> Capacitor_SMD:C_0402_1005Metric
- C16: renamed from C23; footprint Capacitor_SMD:C_0603_1608Metric_Pad1.08x0.95mm_HandSolder -> Capacitor_SMD:C_0402_1005Metric
- C17: renamed from C24; footprint Capacitor_SMD:C_0603_1608Metric_Pad1.08x0.95mm_HandSolder -> Capacitor_SMD:C_0402_1005Metric
- C18: renamed from C25; footprint Capacitor_SMD:C_0603_1608Metric_Pad1.08x0.95mm_HandSolder -> Capacitor_SMD:C_0402_1005Metric
- C19: renamed from C26; footprint Capacitor_SMD:C_0603_1608Metric_Pad1.08x0.95mm_HandSolder -> Capacitor_SMD:C_0402_1005Metric
- C20: renamed from C27; footprint Capacitor_SMD:C_0603_1608Metric_Pad1.08x0.95mm_HandSolder -> Capacitor_SMD:C_0402_1005Metric
- C21: renamed from C28; footprint Capacitor_SMD:C_0603_1608Metric_Pad1.08x0.95mm_HandSolder -> Capacitor_SMD:C_0402_1005Metric
- C22: renamed from C29; footprint Capacitor_SMD:C_0603_1608Metric_Pad1.08x0.95mm_HandSolder -> Capacitor_SMD:C_0402_1005Metric
- C23: renamed from C30; footprint Capacitor_SMD:C_0603_1608Metric_Pad1.08x0.95mm_HandSolder -> Capacitor_SMD:C_0402_1005Metric
- C24: renamed from C31; footprint Capacitor_SMD:C_0603_1608Metric -> Capacitor_SMD:C_0402_1005Metric
- C25: renamed from C32; footprint Capacitor_SMD:C_0603_1608Metric -> Capacitor_SMD:C_0402_1005Metric
- C26: renamed from C33; footprint Capacitor_SMD:C_0603_1608Metric -> Capacitor_SMD:C_0402_1005Metric
- C27: renamed from C34; footprint Capacitor_SMD:C_0603_1608Metric -> Capacitor_SMD:C_0402_1005Metric
- C28: renamed from C35; footprint Capacitor_SMD:C_0603_1608Metric -> Capacitor_SMD:C_0402_1005Metric
- C29: renamed from C36; footprint Capacitor_SMD:C_0603_1608Metric -> Capacitor_SMD:C_0402_1005Metric
- C30: renamed from C37; footprint Capacitor_SMD:C_0603_1608Metric -> Capacitor_SMD:C_0402_1005Metric
- C31: renamed from C38; footprint Capacitor_SMD:C_0603_1608Metric -> Capacitor_SMD:C_0402_1005Metric
- C32: renamed from C39; footprint Capacitor_SMD:C_0603_1608Metric -> Capacitor_SMD:C_0402_1005Metric
- C33: renamed from C40; footprint Capacitor_SMD:C_0603_1608Metric -> Capacitor_SMD:C_0402_1005Metric
- C34: renamed from C41; footprint Capacitor_SMD:C_0603_1608Metric -> Capacitor_SMD:C_0402_1005Metric
- C35: renamed from C42; footprint Capacitor_SMD:C_0603_1608Metric -> Capacitor_SMD:C_0402_1005Metric
- C36: renamed from C43; footprint Capacitor_SMD:C_0603_1608Metric -> Capacitor_SMD:C_0402_1005Metric
- C37: renamed from C44; footprint Capacitor_SMD:C_0603_1608Metric -> Capacitor_SMD:C_0402_1005Metric
- C8: footprint Capacitor_SMD:C_1206_3216Metric_Pad1.33x1.80mm_HandSolder -> Capacitor_SMD:C_0402_1005Metric
- D5, D6, D7, D8, F1: moved to B.Cu
- J13: footprint Connector_PinHeader_1.27mm:PinHeader_2x03_P1.27mm_Vertical -> Tag-Connect:Tag-Connect_TC2030-IDC-NL_2x03_P1.27mm_Vertical
- R1, R10, R11, R12, R13, R14, R15, R16, R17, R18, R19, R2, R20, R21, R22, R23, R24, R3, R4, R5, R6, R7, R8, R9: footprint Resistor_SMD:R_0603_1608Metric_Pad0.98x0.95mm_HandSolder -> FixedTextSizes:R_0402_1005Metric
- R25, R26, R27: footprint Resistor_SMD:R_0603_1608Metric_Pad0.98x0.95mm_HandSolder -> FixedTextSizes:R_0402_1005Metric; moved to B.Cu
- R28: renamed from R30; footprint Resistor_SMD:R_0603_1608Metric_Pad0.98x0.95mm_HandSolder -> FixedTextSizes:R_0402_1005Metric
- R29: renamed from R31; footprint Resistor_SMD:R_0603_1608Metric_Pad0.98x0.95mm_HandSolder -> FixedTextSizes:R_0402_1005Metric
- R30: renamed from R32; footprint Resistor_SMD:R_0603_1608Metric_Pad0.98x0.95mm_HandSolder -> FixedTextSizes:R_0402_1005Metric
- R31: renamed from R33; footprint Resistor_SMD:R_0603_1608Metric_Pad0.98x0.95mm_HandSolder -> FixedTextSizes:R_0402_1005Metric
- R32: renamed from R34; footprint Resistor_SMD:R_0603_1608Metric_Pad0.98x0.95mm_HandSolder -> FixedTextSizes:R_0402_1005Metric
- R33: renamed from R35; footprint Resistor_SMD:R_0603_1608Metric_Pad0.98x0.95mm_HandSolder -> FixedTextSizes:R_0402_1005Metric
- R34: renamed from R36; footprint Resistor_SMD:R_0603_1608Metric_Pad0.98x0.95mm_HandSolder -> FixedTextSizes:R_0402_1005Metric
- R35: renamed from R37; footprint Resistor_SMD:R_0603_1608Metric_Pad0.98x0.95mm_HandSolder -> FixedTextSizes:R_0402_1005Metric
- R36: renamed from R38; footprint Resistor_SMD:R_0603_1608Metric_Pad0.98x0.95mm_HandSolder -> FixedTextSizes:R_0402_1005Metric
- R37: renamed from R39; footprint Resistor_SMD:R_0603_1608Metric_Pad0.98x0.95mm_HandSolder -> FixedTextSizes:R_0402_1005Metric
- R38: renamed from R40; footprint Resistor_SMD:R_1206_3216Metric_Pad1.30x1.75mm_HandSolder -> FixedTextSizes:R_0402_1005Metric
- R39: renamed from R41; footprint Resistor_SMD:R_1206_3216Metric_Pad1.30x1.75mm_HandSolder -> FixedTextSizes:R_0402_1005Metric
- R40: renamed from R42; footprint Resistor_SMD:R_0603_1608Metric_Pad0.98x0.95mm_HandSolder -> FixedTextSizes:R_0402_1005Metric
- R41: renamed from R43; footprint Resistor_SMD:R_0603_1608Metric_Pad0.98x0.95mm_HandSolder -> FixedTextSizes:R_0402_1005Metric
- R42: renamed from R44; footprint Resistor_SMD:R_0603_1608Metric_Pad0.98x0.95mm_HandSolder -> FixedTextSizes:R_0402_1005Metric
- R43: renamed from R45; footprint Resistor_SMD:R_0603_1608Metric_Pad0.98x0.95mm_HandSolder -> FixedTextSizes:R_0402_1005Metric
- R44: renamed from R46; footprint Resistor_SMD:R_0603_1608Metric_Pad0.98x0.95mm_HandSolder -> FixedTextSizes:R_0402_1005Metric
- R45: renamed from R47; footprint Resistor_SMD:R_0603_1608Metric_Pad0.98x0.95mm_HandSolder -> FixedTextSizes:R_0402_1005Metric
- R46: renamed from R48; footprint Resistor_SMD:R_0603_1608Metric_Pad0.98x0.95mm_HandSolder -> FixedTextSizes:R_0402_1005Metric
- R47: renamed from R49; footprint Resistor_SMD:R_0603_1608Metric_Pad0.98x0.95mm_HandSolder -> FixedTextSizes:R_0402_1005Metric
- R48: renamed from R50; footprint Resistor_SMD:R_0603_1608Metric_Pad0.98x0.95mm_HandSolder -> FixedTextSizes:R_0402_1005Metric
- R49: renamed from R51; footprint Resistor_SMD:R_0603_1608Metric_Pad0.98x0.95mm_HandSolder -> FixedTextSizes:R_0402_1005Metric
- R50: renamed from R52; footprint Resistor_SMD:R_0603_1608Metric_Pad0.98x0.95mm_HandSolder -> FixedTextSizes:R_0402_1005Metric
- R51: renamed from R53; footprint Resistor_SMD:R_0603_1608Metric_Pad0.98x0.95mm_HandSolder -> FixedTextSizes:R_0402_1005Metric
- R52: renamed from R54; footprint Resistor_SMD:R_0603_1608Metric_Pad0.98x0.95mm_HandSolder -> FixedTextSizes:R_0402_1005Metric
- R53: renamed from R55; footprint Resistor_SMD:R_0603_1608Metric -> FixedTextSizes:R_0402_1005Metric
- R54: renamed from R56; footprint Resistor_SMD:R_0603_1608Metric -> FixedTextSizes:R_0402_1005Metric
- R55: renamed from R57; footprint Resistor_SMD:R_0603_1608Metric -> FixedTextSizes:R_0402_1005Metric
- R56: renamed from R58; footprint Resistor_SMD:R_0603_1608Metric -> FixedTextSizes:R_0402_1005Metric
- R57: renamed from R59; footprint Resistor_SMD:R_0603_1608Metric -> FixedTextSizes:R_0402_1005Metric
- R58: renamed from R60; footprint Resistor_SMD:R_0603_1608Metric -> FixedTextSizes:R_0402_1005Metric
- R59: renamed from R61; footprint Resistor_SMD:R_0603_1608Metric -> FixedTextSizes:R_0402_1005Metric
- R60: renamed from R62; footprint Resistor_SMD:R_0603_1608Metric -> FixedTextSizes:R_0402_1005Metric
- R61: renamed from R63; footprint Resistor_SMD:R_0603_1608Metric -> FixedTextSizes:R_0402_1005Metric
- R62: renamed from R64; footprint Resistor_SMD:R_0603_1608Metric -> FixedTextSizes:R_0402_1005Metric
- R63: renamed from R65; footprint Resistor_SMD:R_0603_1608Metric -> FixedTextSizes:R_0402_1005Metric
- R64: renamed from R66; footprint Resistor_SMD:R_0603_1608Metric -> FixedTextSizes:R_0402_1005Metric
- R65: renamed from R67; footprint Resistor_SMD:R_0603_1608Metric -> FixedTextSizes:R_0402_1005Metric
- R66: renamed from R68; footprint Resistor_SMD:R_0603_1608Metric -> FixedTextSizes:R_0402_1005Metric
- R67: renamed from R69; footprint Resistor_SMD:R_0603_1608Metric -> FixedTextSizes:R_0402_1005Metric
- R68: renamed from R70; footprint Resistor_SMD:R_0603_1608Metric -> FixedTextSizes:R_0402_1005Metric
- R69: renamed from R71; footprint Resistor_SMD:R_0603_1608Metric -> FixedTextSizes:R_0402_1005Metric
- R70: renamed from R72; footprint Resistor_SMD:R_0603_1608Metric -> FixedTextSizes:R_0402_1005Metric
- R71: renamed from R73; footprint Resistor_SMD:R_0603_1608Metric -> FixedTextSizes:R_0402_1005Metric
- U17: value SN65HVD230 -> TPS562200; footprint Package_SO:SOIC-8_3.9x4.9mm_P1.27mm -> Package_TO_SOT_SMD:SOT-23-6
- moved TP32 145.8 mm to (20.6, 22.4)
- moved R61 142.7 mm to (6.60, 30.7)
- moved J11 134.7 mm to (2.79, 30.0)
- moved JP1 128.3 mm to (27.4, 20.6), turned to 90 degrees
- moved U15 127.8 mm to (11.9, 31.2), turned to 180 degrees
- moved JP2 124.7 mm to (24.4, 20.6), turned to 90 degrees
- moved U17 112.3 mm to (218.8, 138.1)
- moved R71 87.4 mm to (73.9, 29.0), turned to -90 degrees
- moved J13 84.9 mm to (72.4, 25.7), turned to 180 degrees
- moved D7 72.0 mm to (49.0, 22.1)
- moved R27 71.6 mm to (51.0, 19.6), turned to 90 degrees
- moved R26 70.6 mm to (54.4, 19.6), turned to 90 degrees
- moved F1 70.1 mm to (42.2, 16.8), turned to 90 degrees
- moved D8 66.7 mm to (49.0, 24.6), turned to 180 degrees
- moved D18 66.6 mm to (65.8, 66.5), turned to 90 degrees
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- renumbered D11 to D10, D12 to D11, D13 to D12, D14 to D13, D15 to D14, D16 to D15, D17 to D16, D19 to D18, D10 to D9, L2 to L1, U11 to U10, U12 to U11, U13 to U12, U14 to U13, U15 to U14, U16 to U15, U7 to U6, U8 to U7, U9 to U8, U10 to U9
Connections:
- D1 pad 1: +12V -> /Power Supply 1/12V_In_Unprotected
- JP1 pad 2: /Microcontroller/CAN1_H -> /CAN_H
- JP2 pad 2: /Microcontroller/CAN1_L -> /CAN_L
- JP3 pad 1: Net-(D18-Pad3) -> Net-(D17-Pad3)
- JP4 pad 1: Net-(D18-Pad1) -> Net-(D17-Pad1)
- R62 pad 2: Net-(D18-Pad1) -> Net-(D17-Pad1)
- R64 pad 2: Net-(D18-Pad1) -> Net-(D17-Pad1)
- R66 pad 1: Net-(D18-Pad3) -> Net-(D17-Pad3)
- R68 pad 1: Net-(D18-Pad3) -> Net-(D17-Pad3)
- TP31 pad 1: Net-(D18-Pad3) -> Net-(D17-Pad3)
- TP33 pad 1: Net-(D18-Pad1) -> Net-(D17-Pad1)
- U17 pad 1: /Microcontroller/CAN2_TX -> GND
- U17 pad 2: GND -> /Power Supply 1/BUCK/SW
- U17 pad 3: +3V3 -> +12V
- U17 pad 4: /Microcontroller/CAN2_RX -> /Power Supply 1/BUCK/VFB
- U17 pad 5: unconnected-(U17-Pad5) -> /Power Supply 1/BUCK/EN
- U17 pad 6: Net-(D18-Pad1) -> /Power Supply 1/BUCK/VBST
Routing:
- net Net-(D17-Pad4): track 0.00 -> 25.5 mm
- net /IMD_data: track 0.00 -> 24.2 mm, vias 0 -> 1
- net Net-(D17-Pad6): track 0.00 -> 22.8 mm
- net /IMD_fault: track 0.00 -> 22.7 mm, vias 0 -> 1
- net /CAN_H: track 0.00 -> 14.2 mm, vias 0 -> 1
- net /IMD_12V: track 0.00 -> 14.0 mm
- net /CAN_L: track 0.00 -> 13.8 mm
- net GND: track 0.00 -> 13.6 mm, vias 0 -> 6
- net /Microcontroller/SWDIO: track 0.00 -> 11.4 mm
- net /Microcontroller/SWCLK: track 0.00 -> 6.16 mm
- net /IMD_status_output: track 0.00 -> 5.75 mm
- net /IMD_data_low_side: track 0.00 -> 5.47 mm
- net Net-(C34-Pad2): track 0.00 -> 3.62 mm
- net Net-(J13-Pad2): track 0.00 -> 2.26 mm
- added copper zone on In1.Cu, net GND
Other:
- copper layers 2 -> 4

Commit message: More work
Parts:
- D17: moved to B.Cu
- moved R67 150.6 mm to (6.60, 33.5), turned to 180 degrees
- moved R63 142.3 mm to (6.60, 29.2)
- moved R65 138.6 mm to (6.60, 32.0), turned to 180 degrees
- moved C34 137.0 mm to (5.08, 27.2), turned to -90 degrees
- moved R59 92.8 mm to (66.0, 52.6), turned to 90 degrees
- moved R60 87.2 mm to (67.6, 52.6), turned to 90 degrees
- moved D17 86.2 mm to (12.7, 28.7), turned to 90 degrees
- moved D18 10.2 mm to (66.0, 56.4)
Routing:
- net Net-(J11-Pad2): track 0.00 -> 4.95 mm
- net Net-(D17-Pad4): track 25.5 -> 30.4 mm, vias 0 -> 1
- net Net-(D17-Pad6): track 22.8 -> 27.1 mm
- net GND: track 13.6 -> 17.5 mm, vias 6 -> 7
- net Net-(C34-Pad2): track 3.62 -> 7.11 mm
- net Net-(D18-Pad4): track 0.00 -> 1.97 mm
- net Net-(D18-Pad5): track 0.00 -> 1.77 mm

Commit message: More progress
Parts:
- removed D1: D_Schottky, Diode_SMD:D_SMA_Handsoldering
- removed PWR_3V1, PWR_IN1, PWR_IN2: LED, LED_SMD:LED_0603_1608Metric_Pad1.05x0.95mm_HandSolder
- removed PWR_5V1: 100, Resistor_SMD:R_0201_0603Metric_Pad0.64x0.40mm_HandSolder
- added C44: 1uF, FixedTextSizes:C_0603_1608Metric_Pad1.08x0.95mm_HandSolder_Reasonable_Text_Size, F.Cu at (23.2, -59.3)
- added C45: 22uF, FixedTextSizes:C_0603_1608Metric_Pad1.08x0.95mm_HandSolder_Reasonable_Text_Size, F.Cu at (23.2, -61.8)
- added C48: ~, FixedTextSizes:C_0402_1005Metric_Pad0.74x0.62mm_HandSolder_Reasonable_Text_Size, F.Cu at (109.8, -24.6)
- added D21: LED, LED_SMD:LED_0603_1608Metric_Pad1.05x0.95mm_HandSolder, F.Cu at (1.27, 27.3)
- added J13: Conn_01x02, Connector_PinHeader_2.54mm:PinHeader_1x02_P2.54mm_Vertical, F.Cu at (100.5, -13.4)
- added J8: Conn_01x02, Connector_PinHeader_2.54mm:PinHeader_1x02_P2.54mm_Horizontal, F.Cu at (92.0, -25.3)
- added R78: ~, FixedTextSizes:R_0402_1005Metric, F.Cu at (109.8, -26.6)
- added TP42: TestPoint, TestPoint:TestPoint_THTPad_1.0x1.0mm_Drill0.5mm, F.Cu at (58.9, -74.2)
- added TP43: TestPoint, TestPoint:TestPoint_THTPad_1.0x1.0mm_Drill0.5mm, F.Cu at (61.9, -74.2)
- added U16: SN65HVD230, Package_SO:SOIC-8_3.9x4.9mm_P1.27mm, F.Cu at (-13.0, -68.9)
- added U18: AMS1117-3.3, Package_TO_SOT_SMD:SOT-223-3_TabPin2, B.Cu at (9.78, 35.6)
- added U20: LSF0204QPWRQ1, LSF0204QPWRQ1:SOP65P640X120-14N, F.Cu at (151.6, -48.0)
- C1, C10, C11, C12, C13, C14, C15, C16, C17, C19, C2, C20, C21, C22, C23, C24, C25, C26, C27, C28, C29, C3, C30, C31, C32, C33, C34, C35, C36, C37, C4, C5, C6, C7, C8, C9: footprint Capacitor_SMD:C_0402_1005Metric -> FixedTextSizes:C_0402_1005Metric_Pad0.74x0.62mm_HandSolder_Reasonable_Text_Size
- C18: footprint Capacitor_SMD:C_0402_1005Metric -> FixedTextSizes:C_0402_1005Metric_Pad0.74x0.62mm_HandSolder_Reasonable_Text_Size; moved to B.Cu
- C38, C39, C40, C41: footprint Capacitor_SMD:C_0402_1005Metric -> FixedTextSizes:C_0603_1608Metric_Pad1.08x0.95mm_HandSolder_Reasonable_Text_Size; moved to B.Cu
- C42, C43: footprint Capacitor_SMD:C_0402_1005Metric -> FixedTextSizes:C_0603_1608Metric_Pad1.08x0.95mm_HandSolder_Reasonable_Text_Size
- D19: value 20V -> 32V; footprint Diode_SMD:D_0603_1608Metric_Pad1.05x0.95mm_HandSolder -> Diode_SMD:D_SOD-323; moved to B.Cu
- D20: footprint Diode_SMD:D_0603_1608Metric_Pad1.05x0.95mm_HandSolder -> Diode_SMD:D_SMA; moved to B.Cu
- F2: footprint Fuse:Fuse_0603_1608Metric_Pad1.05x0.95mm_HandSolder -> Fuse:Fuse_1206_3216Metric_Pad1.42x1.75mm_HandSolder; moved to B.Cu
- J1: value Conn_01x116 -> Conn_01x20; footprint Connector_Molex:Molex_Micro-Fit_3.0_43045-1600_2x08_P3.00mm_Horizontal -> Connector_Molex:Molex_Micro-Fit_3.0_43045-2000_2x10_P3.00mm_Horizontal
- L2, R38, R39, R40, R41, R42, R43, R44, U10, U8, U9: moved to B.Cu
- R72: value 470 -> 470R; footprint FixedTextSizes:R_0402_1005Metric -> Resistor_SMD:R_0603_1608Metric_Pad0.98x0.95mm_HandSolder
- R73: value 0 -> 10K; footprint FixedTextSizes:R_0402_1005Metric -> Resistor_SMD:R_0603_1608Metric_Pad0.98x0.95mm_HandSolder; moved to B.Cu
- R74: footprint FixedTextSizes:R_0402_1005Metric -> Resistor_SMD:R_0603_1608Metric_Pad0.98x0.95mm_HandSolder
- R75: value 10K -> 54.9K; footprint FixedTextSizes:R_0402_1005Metric -> Resistor_SMD:R_0603_1608Metric_Pad0.98x0.95mm_HandSolder; moved to B.Cu
- R76: value 54.9K -> ~
- U17: value TPS562200 -> LMR51420; moved to B.Cu
- moved R74 304.3 mm to (4.10, -70.8)
- moved C42 302.7 mm to (-0.25, -68.3)
- moved C43 302.7 mm to (-0.25, -70.8)
- moved F2 272.6 mm to (5.84, 11.4)
- moved D20 269.0 mm to (2.79, 17.3), turned to 90 degrees
- moved R72 268.9 mm to (1.27, 31.1), turned to 90 degrees
- moved R73 267.6 mm to (8.89, 19.1)
- moved D19 265.5 mm to (8.89, 15.2)
- moved C40 253.5 mm to (1.91, 22.9), turned to -90 degrees
- moved C39 250.7 mm to (6.35, 17.8), turned to 90 degrees
- moved C38 247.7 mm to (3.81, 22.9), turned to -90 degrees
- moved R75 247.0 mm to (10.2, 29.8), turned to -90 degrees
- moved C41 246.4 mm to (11.4, 26.0)
- moved U17 240.6 mm to (7.62, 22.9)
- moved L2 237.6 mm to (6.35, 28.6), turned to -90 degrees
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- renumbered J9 to J10, J10 to J11, J11 to J12, J13 to J14, J8 to J9
Connections:
- net /IMD_12V renamed /IMD_24V
- net Net-(C8-Pad1) renamed /Precharge_Timer
- net Net-(D19-Pad1) renamed /Power Supply 1/DIODE
- C38 pad 1: +12V -> /Power Supply 1/BUCK/V_in
- C39 pad 1: +12V -> /Power Supply 1/BUCK/V_in
- C40 pad 1: +12V -> /Power Supply 1/BUCK/V_in
- D20 pad 1: +12V -> /Power Supply 1/BUCK/V_in
- F1 pad 1: +12V -> +24V
- F2 pad 2: /Power Supply 1/12V_In_Unprotected -> +24V
- J1 pad 2: /12V_in -> +24V
- JP3 pad 2: /Microcontroller/CAN2_H -> /Telemetry_CAN_H
- JP4 pad 2: /Microcontroller/CAN2_L -> /Telemetry_CAN_L
- R72 pad 1: +12V -> GND
- R73 pad 1: +3V3 -> /Power Supply 1/BUCK/V_in
- R73 pad 2: Net-(PWR_3V1-Pad2) -> /Power Supply 1/BUCK/EN
- R74 pad 1: +12V -> /Power Supply 1/BUCK/VFB
- R74 pad 2: /Power Supply 1/BUCK/EN -> GND
- R75 pad 2: GND -> +5V
- R76 pad 1: /Power Supply 1/BUCK/VFB -> /Watchdog/Microcontroller/I2C1_SDA
- R76 pad 2: +5V -> VDD
- U14 pad 42: /Microcontroller/PA9 -> /Watchdog_RX
- U14 pad 43: /Microcontroller/PA10 -> /Watchdog_TX
- U17 pad 3: +12V -> /Power Supply 1/BUCK/V_in
Routing:
- net /Voltage Measurement/iso_hv_0: track 0.00 -> 32.1 mm
- net /Power Supply 1/BUCK/V_in: track 0.00 -> 19.4 mm, vias 0 -> 1
- net GND: track 17.5 -> 36.2 mm, vias 7 -> 9
- net Net-(R42-Pad1): track 0.00 -> 18.0 mm
- net +5V: track 0.00 -> 17.5 mm
- net /Microcontroller/LED_R: track 0.00 -> 17.4 mm, vias 0 -> 2
- net Net-(R41-Pad1): track 0.00 -> 15.9 mm
- net /Microcontroller/LED_G: track 0.00 -> 14.4 mm, vias 0 -> 2
- net /IMD_24V: track 14.0 -> 0.00 mm
- net /Microcontroller/LED_B: track 0.00 -> 13.8 mm, vias 0 -> 2
- net /Power Supply 1/BUCK/VFB: track 0.00 -> 12.1 mm
- net Net-(D17-Pad6): track 27.1 -> 39.2 mm, vias 0 -> 1
- net /Power Supply 1/BUCK/SW: track 0.00 -> 9.36 mm
- net /Power Supply 1/DIODE: track 0.00 -> 8.61 mm
- net Net-(C21-Pad2): track 0.00 -> 8.60 mm
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- added copper zone on In2.Cu, net GND
- removed copper zone on In1.Cu, net GND
Other:
- board text added: "MCU PWR"
- board text added: "MCU SWD"
- board text added: "Main MCU"
- board text added: "PWR"

Commit message: More work
Parts:
- C13, C16, JP3, JP4, U16: moved to B.Cu
- C18, R40, R41, R42, R43, R44, U10, U8, U9: moved to F.Cu
- moved U11 190.3 mm to (28.1, 49.1)
- moved U12 178.4 mm to (38.9, 49.0)
- moved U13 175.9 mm to (49.8, 49.0)
- moved JP3 116.1 mm to (39.5, 18.2), turned to 90 degrees
- moved JP4 115.5 mm to (36.7, 18.2), turned to 90 degrees
- moved J8 110.3 mm to (2.09, 38.6), turned to 180 degrees
- moved U16 107.0 mm to (38.7, 24.8), turned to 90 degrees
- moved C27 106.8 mm to (60.8, 33.1), turned to 180 degrees
- moved C37 103.9 mm to (57.1, 41.0)
- moved TP15 103.4 mm to (80.9, 31.8)
- moved R70 98.0 mm to (64.3, 27.2)
- moved R69 97.6 mm to (57.1, 42.2), turned to 180 degrees
- moved TP16 97.5 mm to (78.9, 42.2)
- moved R29 97.5 mm to (80.5, 37.1)
- moved R30 95.8 mm to (80.5, 38.5)
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Routing:
- net /Microcontroller/CAN1_TX: track 0.00 -> 59.4 mm
- net /Microcontroller/CAN1_RX: track 0.00 -> 58.8 mm
- net /IMD_fault: track 22.7 -> 71.7 mm
- net /IMD_data: track 24.2 -> 69.3 mm
- net /Shutdown Circuit Control/latch_ready: track 0.00 -> 39.4 mm, vias 0 -> 2
- net Net-(Q11-Pad2): track 0.00 -> 35.8 mm
- net GND: track 36.2 -> 64.7 mm
- net /D_Precharge_cmd: track 0.00 -> 27.9 mm
- net /D_Final_Close_Out: track 0.00 -> 24.9 mm
- net /IMD_24V: track 0.00 -> 19.8 mm
- net +3V3: track 2.77 -> 20.3 mm
- net Net-(R38-Pad2): track 2.23 -> 18.6 mm
- net (no net): track 0.11 -> 16.2 mm
- net /D_IMD_Fault_Latched: track 0.00 -> 14.9 mm
- net /IMD_KE: track 0.00 -> 12.8 mm
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Other:
- board outline added: 140 x 61.5 mm

Commit message: More progress
Parts:
- removed the C13 at (235.2, 65.7)
- removed the C14 at (221.8, 73.4)
- removed the C15 at (227.2, 75.9)
- removed the C16 at (240.4, 64.8)
- removed the C17 at (221.8, 77.7)
- removed the C18 at (227.8, 72.2)
- removed the C19 at (235.2, 69.9)
- removed C2, C3: 22pf, FixedTextSizes:C_0402_1005Metric_Pad0.74x0.62mm_HandSolder_Reasonable_Text_Size
- removed C4, C5: 0.1uf, FixedTextSizes:C_0402_1005Metric_Pad0.74x0.62mm_HandSolder_Reasonable_Text_Size
- removed the C45 at (23.2, -61.8)
- removed the C45 at (238.6, 104.8)
- removed C46: 22uF, Capacitor_SMD:C_0603_1608Metric_Pad1.08x0.95mm_HandSolder
- removed C48: ~, FixedTextSizes:C_0402_1005Metric_Pad0.74x0.62mm_HandSolder_Reasonable_Text_Size
- removed the D9 at (216.2, 67.4)
- removed the D9 at (154.3, -27.1)
- removed the L1 at (149.6, 77.9)
- removed the L1 at (213.8, 75.4)
- removed the R28 at (233.0, 73.3)
- removed the R28 at (161.8, -28.6)
- removed the R29 at (227.0, 78.6)
- removed the R47 at (227.9, 88.8)
- removed the R48 at (232.2, 88.8)
- removed the R49 at (219.4, 95.2)
- removed the R50 at (230.8, 91.3)
- removed TP42, TP43: TestPoint, TestPoint:TestPoint_THTPad_1.0x1.0mm_Drill0.5mm
- removed TP5, TP6: TestPoint, TestPoint:TestPoint_THTPad_D1.0mm_Drill0.5mm
- removed U1: MCP2515-xSO, Package_SO:SOIC-18W_7.5x11.6mm_P1.27mm
- removed U11, U12, U13: LM358, Package_SO:SOIC-8_3.9x4.9mm_P1.27mm
- removed the U18 at (231.4, 107.7)
- removed U2: SN65HVD230, Package_SO:SOIC-8_3.9x4.9mm_P1.27mm
- removed U20: LSF0204QPWRQ1, LSF0204QPWRQ1:SOP65P640X120-14N
- removed the U6 at (227.9, 66.8)
- removed Y1: 16 MHz, Crystal:Crystal_SMD_3225-4Pin_3.2x2.5mm_HandSoldering
- added C45: 22uF, FixedTextSizes:C_0603_1608Metric_Pad1.08x0.95mm_HandSolder_Reasonable_Text_Size, F.Cu at (176.0, -16.4)
- added D9: P6SMB16CA, Diode_SMD:D_SMB_Handsoldering, F.Cu at (164.8, -26.7)
- added L1: 68n, Inductor_SMD:L_0603_1608Metric, F.Cu at (168.6, 116.6)
- added Q13: AO3400A, Package_TO_SOT_SMD:SOT-23, F.Cu at (36.1, 48.8)
- added Q14: AO3400A, Package_TO_SOT_SMD:SOT-23, F.Cu at (40.9, 48.8)
- added Q15: AO3400A, Package_TO_SOT_SMD:SOT-23, F.Cu at (50.7, 48.8)
- added Q16: AO3400A, Package_TO_SOT_SMD:SOT-23, F.Cu at (45.8, 48.8)
- added R28: 10k, FixedTextSizes:R_0402_1005Metric, F.Cu at (171.4, -24.0)
- added R47: 220, FixedTextSizes:R_0402_1005Metric, F.Cu at (189.7, 100.6)
- added R47: 100k, FixedTextSizes:R_0402_1005Metric, F.Cu at (35.2, 45.1)
- added R48: 220, FixedTextSizes:R_0402_1005Metric, F.Cu at (186.8, 104.6)
- added R48: 100k, FixedTextSizes:R_0402_1005Metric, F.Cu at (40.5, 45.3)
- added R49: 220, FixedTextSizes:R_0402_1005Metric, F.Cu at (36.1, 54.2)
- added R49: 220, FixedTextSizes:R_0402_1005Metric, F.Cu at (186.8, 102.6)
- added R50: 220, FixedTextSizes:R_0402_1005Metric, F.Cu at (40.9, 54.4)
- added R50: 220, FixedTextSizes:R_0402_1005Metric, F.Cu at (186.8, 100.6)
- added R77: 10k, FixedTextSizes:R_0402_1005Metric, F.Cu at (46.9, 43.7)
- added R79: 100k, FixedTextSizes:R_0402_1005Metric, F.Cu at (45.1, 45.2)
- C14, C36, C37, R69, Y2: moved to B.Cu
- R4: value 100k -> 10k
- R76: value ~ -> 10k
- R78: value ~ -> 100k
- moved D11 200.0 mm to (36.1, 58.8)
- moved D12 189.2 mm to (41.3, 58.8), turned to 180 degrees
- moved R74 185.5 mm to (184.6, -28.2)
- moved C42 185.5 mm to (180.3, -25.7)
- moved C43 185.5 mm to (180.3, -28.2)
- moved R52 182.6 mm to (45.8, 54.4), turned to -90 degrees
- moved D14 177.3 mm to (51.7, 58.8), turned to 180 degrees
- moved R51 177.0 mm to (50.7, 54.4), turned to -90 degrees
- moved D15 170.1 mm to (46.4, 58.8), turned to 180 degrees
- moved TP1 162.1 mm to (32.6, 53.7)
- moved C44 159.4 mm to (176.0, -13.9)
- moved R4 156.2 mm to (37.0, 43.7), turned to -90 degrees
- moved R5 151.8 mm to (41.9, 43.7), turned to -90 degrees
- moved TP2 146.1 mm to (43.2, 53.8)
- moved TP3 139.4 mm to (53.7, 53.8)
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Connections:
- R4 pad 1: +5V -> /D_AMS_Fault_Latched
- R4 pad 2: /can_~{cs} -> Net-(Q13-Pad1)
- R5 pad 1: +5V -> /D_IMD_Fault_Latched
- R5 pad 2: /can_~{reset} -> Net-(Q14-Pad1)
- R76 pad 1: /Watchdog/Microcontroller/I2C1_SDA -> /D_Precharge_cmd
- R76 pad 2: VDD -> Net-(Q15-Pad1)
- R78 pad 1: Net-(C48-Pad1) -> Net-(Q15-Pad1)
- R78 pad 2: /Watchdog/Vref_A -> GND
- TP1 pad 1: /can_~{cs} -> Net-(Q13-Pad3)
- TP2 pad 1: /can_sck -> Net-(Q14-Pad3)
- TP3 pad 1: /can_miso -> Net-(R51-Pad1)
- TP4 pad 1: /can_mosi -> Net-(R52-Pad1)
Routing:
- net /Microcontroller/CAN2_RX: track 0.00 -> 41.1 mm
- net (no net): track 16.2 -> 0.11 mm
- net /D_Precharge_cmd: track 27.9 -> 19.2 mm
- net Net-(Q13-Pad3): track 0.00 -> 7.44 mm
- net Net-(Q14-Pad3): track 0.00 -> 6.43 mm
- net Net-(R51-Pad1): track 1.27 -> 7.19 mm
- net Net-(Q13-Pad1): track 0.00 -> 5.11 mm
- net Net-(R52-Pad1): track 1.27 -> 6.30 mm
- net Net-(Q16-Pad1): track 0.00 -> 4.93 mm
- net Net-(Q15-Pad1): track 0.00 -> 4.76 mm
- net Net-(D11-Pad2): track 0.00 -> 4.64 mm
- net Net-(Q14-Pad1): track 0.00 -> 4.51 mm
- net Net-(D15-Pad2): track 0.00 -> 4.43 mm
- net Net-(D12-Pad2): track 0.00 -> 4.36 mm
- net GND: track 64.7 -> 69.0 mm
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