File: board/22-ELC-1-01-R1 (TSCU)/20-ELC-1-01-R1.kicad_sch (KiCad schematic)
At the start: 8 parts, among them J1 Conn_01x116, J2 Conn_01x02_Female, J3 Conn_01x06, J4 Conn_01x02, J5 Conn_01x02, J6 Conn_01x06, J7 Conn_01x01

Commit message: More progress
Parts:
- removed D1: D_Schottky, Diode_SMD:D_SMA_Handsoldering, symbol Device:D_Schottky
- added J8: Conn_01x02, Connector_PinHeader_2.54mm:PinHeader_1x02_P2.54mm_Horizontal, symbol Connector_Generic:Conn_01x02
- J1: value Conn_01x116 -> Conn_01x20; footprint Connector_Molex:Molex_Micro-Fit_3.0_43045-1600_2x08_P3.00mm_Horizontal -> Connector_Molex:Molex_Micro-Fit_3.0_43045-2000_2x10_P3.00mm_Horizontal; symbol Connector_Generic:Conn_01x16 -> Connector_Generic:Conn_01x20
Connections:
- net +5V: now also J8.1 (Pin_1)
- net GND: now also J8.2 (Pin_2)
- net 12V_in renamed +24V
- net IMD_12V renamed IMD_24V
- new net Telemetry_CAN_H: J1.17 (Pin_17), J1.19 (Pin_19)
- new net Telemetry_CAN_L: J1.18 (Pin_18), J1.20 (Pin_20)
- no-connect marks 31 -> 27
Other:
- sheet Contactor Logic ports: added Precharge_Timer_Out; removed none
- sheet IMD ports: added 24V_out; removed 12V_out
- sheet Power Supply 1: file ../../2023KicadLibrary/Standardized Subsheets/StandardizedVRMS.kicad_sch -> ../../2023KicadLibrary/Standardized Subsheets/vrmsv2.kicad_sch
- sheet Power Supply 1 ports: added none; removed 12V_In_Unprotected, 12V_Out_Protected, 3V3_Out_Protected, 5V_Out_Protected

Commit message: More progress
Connections:
- no-connect marks 27 -> 26
Other:
- removed sheet CAN
- sheet Indicator LEDs ports: added none; removed AMS_LED_In, IMS_LED_In
