File: board/22-ELC-1-01-R1 (TSCU)/Contactor_Connector.kicad_sch (KiCad schematic)
At the start: 18 parts, among them J8 Conn_02x02_Counter_Clockwise, J9 Conn_02x02_Counter_Clockwise, Q2 2N7002, Q3 CSD18540Q5B

Commit message: Finalized schematic, started board layout
Parts:
- C6, C7: footprint Capacitor_SMD:C_0603_1608Metric_Pad1.08x0.95mm_HandSolder -> Capacitor_SMD:C_0402_1005Metric
- R10, R11, R12, R13, R6, R7, R8, R9: footprint Resistor_SMD:R_0603_1608Metric_Pad0.98x0.95mm_HandSolder -> FixedTextSizes:R_0402_1005Metric
Changed lines of the file:
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@@
   (symbol (lib_id "power:GND") (at 74.93 120.65 0) (unit 1)
     (in_bom yes) (on_board yes)
-    (property "Reference" "#PWR031" (id 0) (at 74.93 127 0)
+    (property "Reference" "#PWR030" (id 0) (at 74.93 127 0)
       (effects (font (size 1.27 1.27)) hide)
     )
@@
       (effects (font (size 1.27 1.27)) (justify left))
     )
-    (property "Footprint" "Resistor_SMD:R_0603_1608Metric_Pad0.98x0.95mm_HandSolder" (id 2) (at 59.69 114.808 90)
+    (property "Footprint" "FixedTextSizes:R_0402_1005Metric" (id 2) (at 59.69 114.808 90)
       (effects (font (size 1.27 1.27)) hide)
     )
@@
     (property "Reference" "R7" (id 0) (at 80.01 101.4222 90))
     (property "Value" "100" (id 1) (at 80.01 103.7336 90))
-    (property "Footprint" "Resistor_SMD:R_0603_1608Metric_Pad0.98x0.95mm_HandSolder" (id 2) (at 80.01 104.902 90)
+    (property "Footprint" "FixedTextSizes:R_0402_1005Metric" (id 2) (at 80.01 104.902 90)
       (effects (font (size 1.27 1.27)) hide)
     )
@@
       (effects (font (size 1.27 1.27)) (justify left))
     )
-    (property "Footprint" "Resistor_SMD:R_0603_1608Metric_Pad0.98x0.95mm_HandSolder" (id 2) (at 90.932 140.97 90)
+    (property "Footprint" "FixedTextSizes:R_0402_1005Metric" (id 2) (at 90.932 140.97 90)
       (effects (font (size 1.27 1.27)) hide)
     )
@@
   (symbol (lib_id "power:GND") (at 92.71 154.94 0) (unit 1)
     (in_bom yes) (on_board yes)
-    (property "Reference" "#PWR033" (id 0) (at 92.71 161.29 0)
+    (property "Reference" "#PWR032" (id 0) (at 92.71 161.29 0)
       (effects (font (size 1.27 1.27)) hide)
     )
@@
     (property "Reference" "R13" (id 0) (at 241.3 88.7222 90))
     (property "Value" "1k" (id 1) (at 241.3 91.0336 90))
-    (property "Footprint" "Resistor_SMD:R_0603_1608Metric_Pad0.98x0.95mm_HandSolder" (id 2) (at 241.3 92.202 90)
+    (property "Footprint" "FixedTextSizes:R_0402_1005Metric" (id 2) (at 241.3 92.202 90)
       (effects (font (size 1.27 1.27)) hide)
     )
@@
   (symbol (lib_id "power:+5V") (at 208.28 97.79 180) (unit 1)
     (in_bom yes) (on_board yes)
-    (property "Reference" "#PWR036" (id 0) (at 208.28 93.98 0)
+    (property "Reference" "#PWR035" (id 0) (at 208.28 93.98 0)
       (effects (font (size 1.27 1.27)) hide)
     )
@@
   (symbol (lib_id "power:+5V") (at 128.905 96.52 0) (unit 1)
     (in_bom yes) (on_board yes)
-    (property "Reference" "#PWR034" (id 0) (at 128.905 100.33 0)
+    (property "Reference" "#PWR033" (id 0) (at 128.905 100.33 0)
       (effects (font (size 1.27 1.27)) hide)
     )
@@
       (effects (font (size 1.27 1.27)) (justify left))
     )
-    (property "Footprint" "Resistor_SMD:R_0603_1608Metric_Pad0.98x0.95mm_HandSolder" (id 2) (at 233.172 97.79 90)
+    (property "Footprint" "FixedTextSizes:R_0402_1005Metric" (id 2) (at 233.172 97.79 90)
       (effects (font (size 1.27 1.27)) hide)
     )
@@
       (effects (font (size 1.27 1.27)) (justify left))
     )
-    (property "Footprint" "Resistor_SMD:R_0603_1608Metric_Pad0.98x0.95mm_HandSolder" (id 2) (at 209.042 91.44 90)
+    (property "Footprint" "FixedTextSizes:R_0402_1005Metric" (id 2) (at 209.042 91.44 90)
       (effects (font (size 1.27 1.27)) hide)
     )
@@
   (symbol (lib_id "power:GND") (at 146.05 83.82 270) (unit 1)
     (in_bom yes) (on_board yes)
-    (property "Reference" "#PWR035" (id 0) (at 139.7 83.82 0)
+    (property "Reference" "#PWR034" (id 0) (at 139.7 83.82 0)
       (effects (font (size 1.27 1.27)) hide)
     )
@@
   (symbol (lib_id "power:GND") (at 212.09 83.82 270) (unit 1)
     (in_bom yes) (on_board yes)
-    (property "Reference" "#PWR037" (id 0) (at 205.74 83.82 0)
+    (property "Reference" "#PWR036" (id 0) (at 205.74 83.82 0)
       (effects (font (size 1.27 1.27)) hide)
     )
@@
       (effects (font (size 1.27 1.27)) (justify right))
     )
-    (property "Footprint" "Capacitor_SMD:C_0603_1608Metric_Pad1.08x0.95mm_HandSolder" (id 2) (at 205.74 91.44 0)
+    (property "Footprint" "Capacitor_SMD:C_0402_1005Metric" (id 2) (at 205.74 91.44 0)
       (effects (font (size 1.27 1.27)) hide)
     )
@@
       (effects (font (size 1.27 1.27)) (justify left))
     )
-    (property "Footprint" "Resistor_SMD:R_0603_1608Metric_Pad0.98x0.95mm_HandSolder" (id 2) (at 143.002 91.44 90)
+    (property "Footprint" "FixedTextSizes:R_0402_1005Metric" (id 2) (at 143.002 91.44 90)
       (effects (font (size 1.27 1.27)) hide)
     )
@@
       (effects (font (size 1.27 1.27)) (justify right))
     )
-    (property "Footprint" "Capacitor_SMD:C_0603_1608Metric_Pad1.08x0.95mm_HandSolder" (id 2) (at 139.7 91.44 0)
+    (property "Footprint" "Capacitor_SMD:C_0402_1005Metric" (id 2) (at 139.7 91.44 0)
       (effects (font (size 1.27 1.27)) hide)
     )
@@
   (symbol (lib_id "power:+5V") (at 87.63 93.98 0) (unit 1)
     (in_bom yes) (on_board yes)
-    (property "Reference" "#PWR032" (id 0) (at 87.63 97.79 0)
+    (property "Reference" "#PWR031" (id 0) (at 87.63 97.79 0)
       (effects (font (size 1.27 1.27)) hide)
     )
@@
       (effects (font (size 1.27 1.27)) (justify left))
     )
-    (property "Footprint" "Resistor_SMD:R_0603_1608Metric_Pad0.98x0.95mm_HandSolder" (id 2) (at 85.852 97.79 90)
-      (effects (font (size 1.27 1.27)) hide)
-    )
+    (property "Footprint" "FixedTextSizes:R_0402_1005Metric" (id 2) (at 85.852 97.79 90)
+      (effects (font (size 1.27 1.27)) hide)
+    )

Commit message: More progress
Parts:
- C6, C7: footprint Capacitor_SMD:C_0402_1005Metric -> FixedTextSizes:C_0402_1005Metric_Pad0.74x0.62mm_HandSolder_Reasonable_Text_Size
- renumbered J9 to J10, J8 to J9
Changed lines of the file:
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@@
   (symbol (lib_id "power:GND") (at 74.93 120.65 0) (unit 1)
     (in_bom yes) (on_board yes)
-    (property "Reference" "#PWR030" (id 0) (at 74.93 127 0)
+    (property "Reference" "#PWR033" (id 0) (at 74.93 127 0)
       (effects (font (size 1.27 1.27)) hide)
     )
@@
   (symbol (lib_id "power:GND") (at 92.71 154.94 0) (unit 1)
     (in_bom yes) (on_board yes)
-    (property "Reference" "#PWR032" (id 0) (at 92.71 161.29 0)
+    (property "Reference" "#PWR035" (id 0) (at 92.71 161.29 0)
       (effects (font (size 1.27 1.27)) hide)
     )
@@
   (symbol (lib_id "power:+5V") (at 208.28 97.79 180) (unit 1)
     (in_bom yes) (on_board yes)
-    (property "Reference" "#PWR035" (id 0) (at 208.28 93.98 0)
+    (property "Reference" "#PWR038" (id 0) (at 208.28 93.98 0)
       (effects (font (size 1.27 1.27)) hide)
     )
@@
   (symbol (lib_id "power:+5V") (at 128.905 96.52 0) (unit 1)
     (in_bom yes) (on_board yes)
-    (property "Reference" "#PWR033" (id 0) (at 128.905 100.33 0)
+    (property "Reference" "#PWR036" (id 0) (at 128.905 100.33 0)
       (effects (font (size 1.27 1.27)) hide)
     )
@@
   (symbol (lib_id "Connector_Generic:Conn_02x02_Counter_Clockwise") (at 151.13 83.82 0) (unit 1)
     (in_bom yes) (on_board yes)
-    (property "Reference" "J8" (id 0) (at 152.4 81.28 0))
+    (property "Reference" "J9" (id 0) (at 152.4 81.28 0))
     (property "Value" "Conn_02x02_Counter_Clockwise" (id 1) (at 152.4 74.93 0)
       (effects (font (size 1.27 1.27)) hide)
@@
   (symbol (lib_id "Connector_Generic:Conn_02x02_Counter_Clockwise") (at 217.17 83.82 0) (unit 1)
     (in_bom yes) (on_board yes)
-    (property "Reference" "J9" (id 0) (at 218.44 81.28 0))
+    (property "Reference" "J10" (id 0) (at 218.44 81.28 0))
     (property "Value" "Conn_02x02_Counter_Clockwise" (id 1) (at 218.44 74.93 0)
       (effects (font (size 1.27 1.27)) hide)
@@
   (symbol (lib_id "power:GND") (at 146.05 83.82 270) (unit 1)
     (in_bom yes) (on_board yes)
-    (property "Reference" "#PWR034" (id 0) (at 139.7 83.82 0)
+    (property "Reference" "#PWR037" (id 0) (at 139.7 83.82 0)
       (effects (font (size 1.27 1.27)) hide)
     )
@@
   (symbol (lib_id "power:GND") (at 212.09 83.82 270) (unit 1)
     (in_bom yes) (on_board yes)
-    (property "Reference" "#PWR036" (id 0) (at 205.74 83.82 0)
+    (property "Reference" "#PWR039" (id 0) (at 205.74 83.82 0)
       (effects (font (size 1.27 1.27)) hide)
     )
@@
       (effects (font (size 1.27 1.27)) (justify right))
     )
-    (property "Footprint" "Capacitor_SMD:C_0402_1005Metric" (id 2) (at 205.74 91.44 0)
+    (property "Footprint" "FixedTextSizes:C_0402_1005Metric_Pad0.74x0.62mm_HandSolder_Reasonable_Text_Size" (id 2) (at 205.74 91.44 0)
       (effects (font (size 1.27 1.27)) hide)
     )
@@
       (effects (font (size 1.27 1.27)) (justify right))
     )
-    (property "Footprint" "Capacitor_SMD:C_0402_1005Metric" (id 2) (at 139.7 91.44 0)
+    (property "Footprint" "FixedTextSizes:C_0402_1005Metric_Pad0.74x0.62mm_HandSolder_Reasonable_Text_Size" (id 2) (at 139.7 91.44 0)
       (effects (font (size 1.27 1.27)) hide)
     )
@@
   (symbol (lib_id "power:+5V") (at 87.63 93.98 0) (unit 1)
     (in_bom yes) (on_board yes)
-    (property "Reference" "#PWR031" (id 0) (at 87.63 97.79 0)
-      (effects (font (size 1.27 1.27)) hide)
-    )
+    (property "Reference" "#PWR034" (id 0) (at 87.63 97.79 0)
+      (effects (font (size 1.27 1.27)) hide)
+    )
