File: board/22-ELC-1-01-R1 (TSCU)/Mounting_Holes_and_Silk.kicad_sch (KiCad schematic)
At the start: 8 parts, among them X1 placeholder_for_picture, X2 placeholder_for_picture

Commit message: All good except need to switch everything to accepting 24v power
Parts:
- X1: footprint LHRE Footprint Library:noidontwantthat -> LHRE Footprint Library:g_noidontwantthat
- X2: footprint LHRE Footprint Library:NewLogo2019 -> LHRE Footprint Library:logo_lhr
Changed lines of the file:
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@@
     (property "Reference" "X1" (id 0) (at 180.34 103.759 0))
     (property "Value" "placeholder_for_picture" (id 1) (at 180.34 106.0704 0))
-    (property "Footprint" "LHRE Footprint Library:noidontwantthat" (id 2) (at 179.07 99.06 0)
+    (property "Footprint" "LHRE Footprint Library:g_noidontwantthat" (id 2) (at 179.07 99.06 0)
       (effects (font (size 1.27 1.27)) hide)
     )
@@
     (property "Reference" "X2" (id 0) (at 180.34 115.189 0))
     (property "Value" "placeholder_for_picture" (id 1) (at 180.34 117.5004 0))
-    (property "Footprint" "LHRE Footprint Library:NewLogo2019" (id 2) (at 179.07 110.49 0)
+    (property "Footprint" "LHRE Footprint Library:logo_lhr" (id 2) (at 179.07 110.49 0)
       (effects (font (size 1.27 1.27)) hide)
     )
