File: board/22-ELC-1-01-R1 (TSCU)/shutdown_circuit_switch_bms.kicad_sch (KiCad schematic)
At the start: 7 parts, among them Q1 AO3400A

Commit message: More progress
Parts:
- C1: footprint Capacitor_SMD:C_0402_1005Metric -> FixedTextSizes:C_0402_1005Metric_Pad0.74x0.62mm_HandSolder_Reasonable_Text_Size
Changed lines of the file:
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@@
   (symbol (lib_id "power:+5V") (at 50.8 88.9 0) (unit 1)
     (in_bom yes) (on_board yes)
-    (property "Reference" "#PWR011" (id 0) (at 50.8 92.71 0)
+    (property "Reference" "#PWR014" (id 0) (at 50.8 92.71 0)
       (effects (font (size 1.27 1.27)) hide)
     )
@@
       (effects (font (size 1.27 1.27)) (justify left))
     )
-    (property "Footprint" "Capacitor_SMD:C_0402_1005Metric" (id 2) (at 89.8652 100.33 0)
+    (property "Footprint" "FixedTextSizes:C_0402_1005Metric_Pad0.74x0.62mm_HandSolder_Reasonable_Text_Size" (id 2) (at 89.8652 100.33 0)
       (effects (font (size 1.27 1.27)) hide)
     )
@@
   (symbol (lib_id "power:GND") (at 88.9 100.33 0) (unit 1)
     (in_bom yes) (on_board yes)
-    (property "Reference" "#PWR014" (id 0) (at 88.9 106.68 0)
+    (property "Reference" "#PWR017" (id 0) (at 88.9 106.68 0)
       (effects (font (size 1.27 1.27)) hide)
     )
@@
   (symbol (lib_id "power:GND") (at 107.95 104.14 0) (unit 1)
     (in_bom yes) (on_board yes)
-    (property "Reference" "#PWR016" (id 0) (at 107.95 110.49 0)
+    (property "Reference" "#PWR019" (id 0) (at 107.95 110.49 0)
       (effects (font (size 1.27 1.27)) hide)
     )
@@
   (symbol (lib_id "power:+5V") (at 107.95 80.01 0) (unit 1)
     (in_bom yes) (on_board yes)
-    (property "Reference" "#PWR015" (id 0) (at 107.95 83.82 0)
+    (property "Reference" "#PWR018" (id 0) (at 107.95 83.82 0)
       (effects (font (size 1.27 1.27)) hide)
     )
@@
   (symbol (lib_id "power:GND") (at 64.77 120.65 0) (unit 1)
     (in_bom yes) (on_board yes)
-    (property "Reference" "#PWR013" (id 0) (at 64.77 127 0)
+    (property "Reference" "#PWR016" (id 0) (at 64.77 127 0)
       (effects (font (size 1.27 1.27)) hide)
     )
@@
   (symbol (lib_id "power:+5V") (at 64.77 81.28 0) (unit 1)
     (in_bom yes) (on_board yes)
-    (property "Reference" "#PWR012" (id 0) (at 64.77 85.09 0)
+    (property "Reference" "#PWR015" (id 0) (at 64.77 85.09 0)
       (effects (font (size 1.27 1.27)) hide)
     )
